File: HW/Mainboard/v0.1/mainboard.kicad_sch (KiCad schematic)
At the start: 0 parts

Commit message: New footprint and symbol for 386
Parts:
- added U1: ~, symbol 386_kicad_lib:80386DX

Commit message: new
Parts:
- removed U1: ~, symbol 386_kicad_lib:80386DX
